File: KiCad/motor_driver.sch (KiCad schematic (older format))
At the start: 17 parts, among them J1 sig_m1, J10 m4, J11 m5, J12 m6, J13 Conn_01x03, J14 power12v, J2 sig_m2, J3 sig_m3, J4 sig_m4, J5 sig_m5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

Commit message: one f*** layer pcb finished, with just 3 bridges
Parts:
- removed U2, U3: L293D, Housings_DIP:DIP-16_W7.62mm_Socket_LongPads, symbol L293D
- added U2, U3: L293D, Housings_DIP:DIP-16_W7.62mm_Socket_LongPads, symbol L293D
- J1: value sig_m1 -> Conn_01x02
- J2: value sig_m2 -> Conn_01x02
- J3: value sig_m3 -> Conn_01x02
- J4: value sig_m4 -> Conn_01x02
- J5: value sig_m5 -> Conn_01x02
- J6: value sig_m6 -> Conn_01x02
Connections:
- wire segments 12 -> 6
Other:
- moved on the sheet: J10, J11, J12, J14, J7, J8, J9
