File: Hardware/KiCad/motor_driver.sch (KiCad schematic (older format))
At the start: 17 parts, among them J1 Conn_01x02, J10 m4, J11 m5, J12 m6, J13 Conn_01x03, J14 power12v, J2 Conn_01x02, J3 Conn_01x02, J4 Conn_01x02, J5 Conn_01x02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

Commit message: motor driver pcb mkII
Parts:
- added J15, J16: Conn_01x01, Pin_Headers:Pin_Header_Straight_1x01_Pitch2.00mm, symbol Conn_01x01
Connections:
- net GND: now also J16.1 (Pin_1)
- net ardu5V: now also J15.1 (Pin_1)
Other:
- note added: "These connectors are used to 'bridge' with wires bc we dont have 2 layers"
- moved on the sheet: J1, J10, J11, J12, J13, J14, J2, J3, J4, J5, J6, J7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
